Commit message: Rebase from 'release/rolling/ur_description'

File: urdf/ur.ros2_control.xacro (robot description, xacro)
@@ -3,5 +3,4 @@
   <xacro:macro name="ur_ros2_control" params="
     name
-    prefix
     use_fake_hardware:=false fake_sensor_commands:=false
     sim_gazebo:=false
@@ -13,10 +12,14 @@
     input_recipe_filename tf_prefix
     hash_kinematics robot_ip
-    tool_voltage:=24 tool_parity:=0 tool_baud_rate:=115200 tool_stop_bits:=1
+    tool_voltage:=0 tool_parity:=0 tool_baud_rate:=115200 tool_stop_bits:=1
     tool_rx_idle_chars:=1.5 tool_tx_idle_chars:=3.5 tool_device_name:=/tmp/ttyUR tool_tcp_port:=54321
     reverse_port:=50001
     script_sender_port:=50002
     reverse_ip:=0.0.0.0
-    script_command_port:=50004">
+    script_command_port:=50004
+    trajectory_port:=50003
+    non_blocking_read:=false
+    keep_alive_count:=2
+    ">
     <ros2_control name="${name}" type="system">
       <hardware>
@@ -43,6 +46,7 @@
           <param name="reverse_ip">${reverse_ip}</param>
           <param name="script_command_port">${script_command_port}</param>
-          <param name="tf_prefix">"${tf_prefix}"</param>
-          <param name="non_blocking_read">0</param>
+          <param name="trajectory_port">${trajectory_port}</param>
+          <param name="tf_prefix">${tf_prefix}</param>
+          <param name="non_blocking_read">${non_blocking_read}</param>
           <param name="servoj_gain">2000</param>
           <param name="servoj_lookahead_time">0.03</param>
@@ -57,7 +61,8 @@
           <param name="tool_device_name">${tool_device_name}</param>
           <param name="tool_tcp_port">${tool_tcp_port}</param>
+          <param name="keep_alive_count">${keep_alive_count}</param>
         </xacro:unless>
       </hardware>
-      <joint name="${prefix}shoulder_pan_joint">
+      <joint name="${tf_prefix}shoulder_pan_joint">
         <command_interface name="position">
           <param name="min">{-2*pi}</param>
@@ -75,5 +80,5 @@
         <state_interface name="effort"/>
       </joint>
-      <joint name="${prefix}shoulder_lift_joint">
+      <joint name="${tf_prefix}shoulder_lift_joint">
         <command_interface name="position">
           <param name="min">{-2*pi}</param>
@@ -91,5 +96,5 @@
         <state_interface name="effort"/>
       </joint>
-      <joint name="${prefix}elbow_joint">
+      <joint name="${tf_prefix}elbow_joint">
         <command_interface name="position">
           <param name="min">{-pi}</param>
@@ -107,5 +112,5 @@
         <state_interface name="effort"/>
       </joint>
-      <joint name="${prefix}wrist_1_joint">
+      <joint name="${tf_prefix}wrist_1_joint">
         <command_interface name="position">
           <param name="min">{-2*pi}</param>
@@ -123,5 +128,5 @@
         <state_interface name="effort"/>
       </joint>
-      <joint name="${prefix}wrist_2_joint">
+      <joint name="${tf_prefix}wrist_2_joint">
         <command_interface name="position">
           <param name="min">{-2*pi}</param>
@@ -139,5 +144,5 @@
         <state_interface name="effort"/>
       </joint>
-      <joint name="${prefix}wrist_3_joint">
+      <joint name="${tf_prefix}wrist_3_joint">
         <command_interface name="position">
           <param name="min">{-2*pi}</param>
@@ -156,5 +161,5 @@
       </joint>
       <xacro:unless value="${sim_gazebo or sim_ignition}">
-        <sensor name="tcp_fts_sensor">
+        <sensor name="${tf_prefix}tcp_fts_sensor">
           <state_interface name="force.x"/>
           <state_interface name="force.y"/>
@@ -165,5 +170,5 @@
         </sensor>
         <!-- NOTE The following are joints used only for testing with fake hardware and will change in the future -->
-        <gpio name="speed_scaling">
+        <gpio name="${tf_prefix}speed_scaling">
           <state_interface name="speed_scaling_factor"/>
           <param name="initial_speed_scaling_factor">1</param>
@@ -171,5 +176,5 @@
           <command_interface name="target_speed_fraction_async_success"/>
         </gpio>
-        <gpio name="gpio">
+        <gpio name="${tf_prefix}gpio">
           <command_interface name="standard_digital_output_cmd_0"/>
           <command_interface name="standard_digital_output_cmd_1"/>
@@ -265,5 +270,5 @@
           <state_interface name="program_running"/>
         </gpio>
-        <gpio name="payload">
+        <gpio name="${tf_prefix}payload">
           <command_interface name="mass"/>
           <command_interface name="cog.x"/>
@@ -272,13 +277,17 @@
           <command_interface name="payload_async_success"/>
         </gpio>
-        <gpio name="resend_robot_program">
+        <gpio name="${tf_prefix}resend_robot_program">
           <command_interface name="resend_robot_program_cmd"/>
           <command_interface name="resend_robot_program_async_success"/>
         </gpio>
-        <gpio name="zero_ftsensor">
+        <gpio name="${tf_prefix}hand_back_control">
+          <command_interface name="hand_back_control_cmd"/>
+          <command_interface name="hand_back_control_async_success"/>
+        </gpio>
+        <gpio name="${tf_prefix}zero_ftsensor">
           <command_interface name="zero_ftsensor_cmd"/>
           <command_interface name="zero_ftsensor_async_success"/>
         </gpio>
-        <gpio name="system_interface">
+        <gpio name="${tf_prefix}system_interface">
           <state_interface name="initialized"/>
         </gpio>

File: urdf/ur.urdf.xacro (robot description, xacro)
@@ -9,5 +9,5 @@
    <xacro:arg name="ur_type" default="ur5x"/>
    <!-- parameters -->
-   <xacro:arg name="prefix" default="" />
+   <xacro:arg name="tf_prefix" default="" />
    <xacro:arg name="joint_limit_params" default="$(find ur_description)/config/$(arg ur_type)/joint_limits.yaml"/>
    <xacro:arg name="kinematics_params" default="$(find ur_description)/config/$(arg ur_type)/default_kinematics.yaml"/>
@@ -28,5 +28,5 @@
    <!--   tool communication related parameters-->
    <xacro:arg name="use_tool_communication" default="false" />
-   <xacro:arg name="tool_voltage" default="24" />
+   <xacro:arg name="tool_voltage" default="0" />
    <xacro:arg name="tool_parity" default="0" />
    <xacro:arg name="tool_baud_rate" default="115200" />
@@ -51,5 +51,5 @@
    <xacro:ur_robot
      name="$(arg name)"
-     prefix="$(arg prefix)"
+     tf_prefix="$(arg tf_prefix)"
      parent="world"
      joint_limits_parameters_file="$(arg joint_limit_params)"
@@ -102,5 +102,5 @@
       <plugin filename="libign_ros2_control-system.so" name="ign_ros2_control::IgnitionROS2ControlPlugin">
         <parameters>$(arg simulation_controllers)</parameters>
-        <controller_manager_node_name>$(arg prefix)controller_manager</controller_manager_node_name>
+        <controller_manager_node_name>$(arg tf_prefix)controller_manager</controller_manager_node_name>
       </plugin>
     </gazebo>

File: urdf/ur_macro.xacro (robot description, xacro)
@@ -46,5 +46,5 @@
   <xacro:macro name="ur_robot" params="
     name
-    prefix
+    tf_prefix
     parent
     *origin
@@ -64,5 +64,5 @@
     initial_positions:=${dict(shoulder_pan_joint=0.0,shoulder_lift_joint=-1.57,elbow_joint=0.0,wrist_1_joint=-1.57,wrist_2_joint=0.0,wrist_3_joint=0.0)}
     use_tool_communication:=false
-    tool_voltage:=24
+    tool_voltage:=0
     tool_parity:=0
     tool_baud_rate:=115200
@@ -79,5 +79,9 @@
     script_sender_port:=50002
     reverse_ip:=0.0.0.0
-    script_command_port:=50004">
+    script_command_port:=50004
+    trajectory_port:=50003
+    non_blocking_read:=false
+    keep_alive_count:=2"
+    >
     <!-- Load configuration data from the provided .yaml files -->
     <xacro:read_model_data
@@ -91,5 +95,5 @@
     <!-- ros2 control instance -->
     <xacro:ur_ros2_control
-      name="${name}" prefix="${prefix}"
+      name="${name}"
       use_fake_hardware="${use_fake_hardware}"
       initial_positions="${initial_positions}"
@@ -101,5 +105,5 @@
       output_recipe_filename="${output_recipe_filename}"
       input_recipe_filename="${input_recipe_filename}"
-      tf_prefix=""
+      tf_prefix="${tf_prefix}"
       hash_kinematics="${kinematics_hash}"
       robot_ip="${robot_ip}"
@@ -117,4 +121,7 @@
       reverse_ip="${reverse_ip}"
       script_command_port="${script_command_port}"
+      trajectory_port="${trajectory_port}"
+      non_blocking_read="${non_blocking_read}"
+      keep_alive_count="${keep_alive_count}"
       />
     <!-- Add URDF transmission elements (for ros_control) -->
@@ -122,6 +129,6 @@
     <!-- Placeholder for ros2_control transmission which don't yet exist -->
     <!-- links -  main serial chain -->
-    <link name="${prefix}base_link"/>
-    <link name="${prefix}base_link_inertia">
+    <link name="${tf_prefix}base_link"/>
+    <link name="${tf_prefix}base_link_inertia">
       <visual>
         <origin xyz="0 0 0" rpy="0 0 ${pi}"/>
@@ -140,5 +147,5 @@
       </xacro:cylinder_inertial>
     </link>
-    <link name="${prefix}shoulder_link">
+    <link name="${tf_prefix}shoulder_link">
       <visual>
         <origin xyz="0 0 0" rpy="0 0 ${pi}"/>
@@ -157,5 +164,5 @@
       </xacro:cylinder_inertial>
     </link>
-    <link name="${prefix}upper_arm_link">
+    <link name="${tf_prefix}upper_arm_link">
       <visual>
         <origin xyz="0 0 ${shoulder_offset}" rpy="${pi/2} 0 ${-pi/2}"/>
@@ -174,5 +181,5 @@
       </xacro:cylinder_inertial>
     </link>
-    <link name="${prefix}forearm_link">
+    <link name="${tf_prefix}forearm_link">
       <visual>
         <origin xyz="0 0 ${elbow_offset}" rpy="${pi/2} 0 ${-pi/2}"/>
@@ -191,5 +198,5 @@
       </xacro:cylinder_inertial>
     </link>
-    <link name="${prefix}wrist_1_link">
+    <link name="${tf_prefix}wrist_1_link">
 	  <xacro:get_visual_params name="wrist_1" type="visual_offset"/>
       <visual>
@@ -209,5 +216,5 @@
       </xacro:cylinder_inertial>
     </link>
-    <link name="${prefix}wrist_2_link">
+    <link name="${tf_prefix}wrist_2_link">
 	  <xacro:get_visual_params name="wrist_2" type="visual_offset"/>
       <visual>
@@ -227,5 +234,5 @@
       </xacro:cylinder_inertial>
     </link>
-    <link name="${prefix}wrist_3_link">
+    <link name="${tf_prefix}wrist_3_link">
 	  <xacro:get_visual_params name="wrist_3" type="visual_offset"/>
       <visual>
@@ -246,13 +253,13 @@
     </link>
     <!-- base_joint fixes base_link to the environment -->
-    <joint name="${prefix}base_joint" type="fixed">
+    <joint name="${tf_prefix}base_joint" type="fixed">
       <xacro:insert_block name="origin" />
       <parent link="${parent}" />
-      <child link="${prefix}base_link" />
+      <child link="${tf_prefix}base_link" />
     </joint>
     <!-- joints - main serial chain -->
-    <joint name="${prefix}base_link-base_link_inertia" type="fixed">
-      <parent link="${prefix}base_link" />
-      <child link="${prefix}base_link_inertia" />
+    <joint name="${tf_prefix}base_link-base_link_inertia" type="fixed">
+      <parent link="${tf_prefix}base_link" />
+      <child link="${tf_prefix}base_link_inertia" />
       <!-- 'base_link' is REP-103 aligned (so X+ forward), while the internal
            frames of the robot/controller have X+ pointing backwards.
@@ -262,7 +269,7 @@
       <origin xyz="0 0 0" rpy="0 0 ${pi}" />
     </joint>
-    <joint name="${prefix}shoulder_pan_joint" type="revolute">
-      <parent link="${prefix}base_link_inertia" />
-      <child link="${prefix}shoulder_link" />
+    <joint name="${tf_prefix}shoulder_pan_joint" type="revolute">
+      <parent link="${tf_prefix}base_link_inertia" />
+      <child link="${tf_prefix}shoulder_link" />
       <origin xyz="${shoulder_x} ${shoulder_y} ${shoulder_z}" rpy="${shoulder_roll} ${shoulder_pitch} ${shoulder_yaw}" />
       <axis xyz="0 0 1" />
@@ -274,7 +281,7 @@
       <dynamics damping="0" friction="0"/>
     </joint>
-    <joint name="${prefix}shoulder_lift_joint" type="revolute">
-      <parent link="${prefix}shoulder_link" />
-      <child link="${prefix}upper_arm_link" />
+    <joint name="${tf_prefix}shoulder_lift_joint" type="revolute">
+      <parent link="${tf_prefix}shoulder_link" />
+      <child link="${tf_prefix}upper_arm_link" />
       <origin xyz="${upper_arm_x} ${upper_arm_y} ${upper_arm_z}" rpy="${upper_arm_roll} ${upper_arm_pitch} ${upper_arm_yaw}" />
       <axis xyz="0 0 1" />
@@ -286,7 +293,7 @@
       <dynamics damping="0" friction="0"/>
     </joint>
-    <joint name="${prefix}elbow_joint" type="revolute">
-      <parent link="${prefix}upper_arm_link" />
-      <child link="${prefix}forearm_link" />
+    <joint name="${tf_prefix}elbow_joint" type="revolute">
+      <parent link="${tf_prefix}upper_arm_link" />
+      <child link="${tf_prefix}forearm_link" />
       <origin xyz="${forearm_x} ${forearm_y} ${forearm_z}" rpy="${forearm_roll} ${forearm_pitch} ${forearm_yaw}" />
       <axis xyz="0 0 1" />
@@ -298,7 +305,7 @@
       <dynamics damping="0" friction="0"/>
     </joint>
-    <joint name="${prefix}wrist_1_joint" type="revolute">
-      <parent link="${prefix}forearm_link" />
-      <child link="${prefix}wrist_1_link" />
+    <joint name="${tf_prefix}wrist_1_joint" type="revolute">
+      <parent link="${tf_prefix}forearm_link" />
+      <child link="${tf_prefix}wrist_1_link" />
       <origin xyz="${wrist_1_x} ${wrist_1_y} ${wrist_1_z}" rpy="${wrist_1_roll} ${wrist_1_pitch} ${wrist_1_yaw}" />
       <axis xyz="0 0 1" />
@@ -310,7 +317,7 @@
       <dynamics damping="0" friction="0"/>
     </joint>
-    <joint name="${prefix}wrist_2_joint" type="revolute">
-      <parent link="${prefix}wrist_1_link" />
-      <child link="${prefix}wrist_2_link" />
+    <joint name="${tf_prefix}wrist_2_joint" type="revolute">
+      <parent link="${tf_prefix}wrist_1_link" />
+      <child link="${tf_prefix}wrist_2_link" />
       <origin xyz="${wrist_2_x} ${wrist_2_y} ${wrist_2_z}" rpy="${wrist_2_roll} ${wrist_2_pitch} ${wrist_2_yaw}" />
       <axis xyz="0 0 1" />
@@ -322,7 +329,7 @@
       <dynamics damping="0" friction="0"/>
     </joint>
-    <joint name="${prefix}wrist_3_joint" type="revolute">
-      <parent link="${prefix}wrist_2_link" />
-      <child link="${prefix}wrist_3_link" />
+    <joint name="${tf_prefix}wrist_3_joint" type="revolute">
+      <parent link="${tf_prefix}wrist_2_link" />
+      <child link="${tf_prefix}wrist_3_link" />
       <origin xyz="${wrist_3_x} ${wrist_3_y} ${wrist_3_z}" rpy="${wrist_3_roll} ${wrist_3_pitch} ${wrist_3_yaw}" />
       <axis xyz="0 0 1" />
@@ -334,13 +341,13 @@
       <dynamics damping="0" friction="0"/>
     </joint>
-    <link name="${prefix}ft_frame"/>
-    <joint name="${prefix}wrist_3_link-ft_frame" type="fixed">
-      <parent link="${prefix}wrist_3_link"/>
-      <child link="${prefix}ft_frame"/>
+    <link name="${tf_prefix}ft_frame"/>
+    <joint name="${tf_prefix}wrist_3_link-ft_frame" type="fixed">
+      <parent link="${tf_prefix}wrist_3_link"/>
+      <child link="${tf_prefix}ft_frame"/>
       <origin xyz="0 0 0" rpy="${pi} 0 0"/>
     </joint>
     <!-- ROS-Industrial 'base' frame - base_link to UR 'Base' Coordinates transform -->
-    <link name="${prefix}base"/>
-    <joint name="${prefix}base_link-base_fixed_joint" type="fixed">
+    <link name="${tf_prefix}base"/>
+    <joint name="${tf_prefix}base_link-base_fixed_joint" type="fixed">
       <!-- Note the rotation over Z of pi radians - as base_link is REP-103
            aligned (i.e., has X+ forward, Y+ left and Z+ up), this is needed
@@ -349,21 +356,21 @@
       -->
       <origin xyz="0 0 0" rpy="0 0 ${pi}"/>
-      <parent link="${prefix}base_link"/>
-      <child link="${prefix}base"/>
+      <parent link="${tf_prefix}base_link"/>
+      <child link="${tf_prefix}base"/>
     </joint>
     <!-- ROS-Industrial 'flange' frame - attachment point for EEF models -->
-    <link name="${prefix}flange" />
-    <joint name="${prefix}wrist_3-flange" type="fixed">
-      <parent link="${prefix}wrist_3_link" />
-      <child link="${prefix}flange" />
+    <link name="${tf_prefix}flange" />
+    <joint name="${tf_prefix}wrist_3-flange" type="fixed">
+      <parent link="${tf_prefix}wrist_3_link" />
+      <child link="${tf_prefix}flange" />
       <origin xyz="0 0 0" rpy="0 ${-pi/2.0} ${-pi/2.0}" />
     </joint>
     <!-- ROS-Industrial 'tool0' frame - all-zeros tool frame -->
-    <link name="${prefix}tool0"/>
-    <joint name="${prefix}flange-tool0" type="fixed">
+    <link name="${tf_prefix}tool0"/>
+    <joint name="${tf_prefix}flange-tool0" type="fixed">
       <!-- default toolframe - X+ left, Y+ up, Z+ front -->
       <origin xyz="0 0 0" rpy="${pi/2.0} 0 ${pi/2.0}"/>
-      <parent link="${prefix}flange"/>
-      <child link="${prefix}tool0"/>
+      <parent link="${tf_prefix}flange"/>
+      <child link="${tf_prefix}tool0"/>
     </joint>
   </xacro:macro>
